File: pcb/manaita.kicad_pcb (KiCad board)
At the start: 2 copper layers, 107 parts, among them J1 SCK, J2 RST, J3 MOSI, J4 MISO, J5 VCC, J6 GND, U1 ATmega32U4, Y1 Crystal

Commit message: WIP
Parts:
- added J4: Conn_01x01, swanmatch:M2hole, F.Cu at (226.2, 83.3)
- added J4: Conn_01x01, swanmatch:M2hole, F.Cu at (54.8, 83.3)
- added J4: Conn_01x01, swanmatch:M2hole, F.Cu at (159.5, 64.3)
- added J4: Conn_01x01, swanmatch:M2hole, F.Cu at (121.4, 64.3)
- added J4: Conn_01x01, swanmatch:M2hole, F.Cu at (250.0, 45.2)
- added J4: Conn_01x01, swanmatch:M2hole, F.Cu at (40.5, 45.2)
- added Ref**: Val**, swanmatch:SpacerHole, F.Cu at (64.3, 83.8)
- added Ref**: Val**, swanmatch:SpacerHole, F.Cu at (140.5, 63.8)
- added Ref**: Val**, swanmatch:SpacerHole, F.Cu at (216.7, 83.8)
- added Ref**: Val**, swanmatch:SpacerHole, F.Cu at (231.0, 44.7)
- added Ref**: Val**, swanmatch:SpacerHole, F.Cu at (59.5, 44.7)
- U1: value ATmega32U4 -> ATmega32U4-AU
- USB1: footprint Connector_PinHeader_2.54mm:PinHeader_1x04_P2.54mm_Horizontal -> Connector_JST:JST_EH_S4B-EH_1x04_P2.50mm_Horizontal
- moved R4 23.4 mm to (59.8, 95.3), turned to 0 degrees
- moved C7 20.4 mm to (56.8, 88.8)
- moved C6 12.9 mm to (54.3, 88.8)
- moved J5 12.8 mm to (43.8, 99.8)
- moved C3 12.8 mm to (59.8, 99.3), turned to 180 degrees
- moved J4 12.3 mm to (41.8, 99.8)
- moved R1 11.9 mm to (62.8, 90.3), turned to 180 degrees
- moved J1 11.8 mm to (39.8, 99.8)
- moved J2 11.3 mm to (37.8, 99.8)
- moved J3 10.8 mm to (35.8, 99.8)
- moved USB1 10.8 mm to (42.8, 86.8), turned to 270 degrees
- moved J6 10.3 mm to (33.8, 99.8)
- moved SW_RESET1 10.3 mm to (26.8, 99.8)
- moved R3 10.2 mm to (51.7, 94.3), turned to 180 degrees
- moved R2 6.81 mm to (51.7, 98.3), turned to 180 degrees
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Connections:
- U1 pad 1: (no net) -> Net-(U1-Pad1)
- U1 pad 18: (no net) -> Net-(U1-Pad18)
- U1 pad 19: (no net) -> Net-(U1-Pad19)
- U1 pad 22: (no net) -> Net-(U1-Pad22)
- U1 pad 26: (no net) -> Net-(U1-Pad26)
- U1 pad 27: (no net) -> Net-(U1-Pad27)
- U1 pad 40: (no net) -> Net-(U1-Pad40)
- U1 pad 41: (no net) -> Net-(U1-Pad41)
- U1 pad 42: (no net) -> Net-(U1-Pad42)
Routing:
- net GND: track 0.00 -> 139.6 mm
- net +5V: track 0.00 -> 139.5 mm
- net Net-(R2-Pad1): track 0.00 -> 29.3 mm, vias 0 -> 2
- net Net-(R3-Pad1): track 0.00 -> 27.9 mm, vias 0 -> 2
- net D+: track 0.00 -> 10.1 mm
- net D-: track 0.00 -> 9.47 mm
Other:
- board outline added: 267.7 x 100.7 mm
- net class GND added: clearance 0.2, trace_width 0.3, via_dia 0.8, via_drill 0.4
- net class VCC added: clearance 0.2, trace_width 0.3, via_dia 0.8, via_drill 0.4

Commit message: :construction: (all) WIP
Parts:
- removed the J4 at (226.2, 83.3)
- removed the J4 at (54.8, 83.3)
- removed the J4 at (159.5, 64.3)
- removed the J4 at (121.4, 64.3)
- removed the J4 at (250.0, 45.2)
- removed Ref** (x5): Val**, swanmatch:SpacerHole
- added D42: D_Zener, Diode_SMD:D_SOD-123, F.Cu at (77.2, 21.4)
- added D43: D_Zener, Diode_SMD:D_SOD-123, F.Cu at (77.2, 25.1)
- added F1: 500mA, Fuse:Fuse_0805_2012Metric_Pad1.15x1.40mm_HandSolder, F.Cu at (71.1, 18.6)
- added JH2: Conn_01x01, swanmatch:M2hole, F.Cu at (250.0, 45.2)
- added JH3: Conn_01x01, swanmatch:M2hole, F.Cu at (121.4, 64.3)
- added JH4: Conn_01x01, swanmatch:M2hole, F.Cu at (159.5, 64.3)
- added JH5: Conn_01x01, swanmatch:M2hole, F.Cu at (54.8, 83.3)
- added JH6: Conn_01x01, swanmatch:M2hole, F.Cu at (226.2, 83.3)
- added RefH1: Val**, swanmatch:SpacerHole, F.Cu at (59.5, 44.7)
- added RefH2: Val**, swanmatch:SpacerHole, F.Cu at (231.0, 44.7)
- added RefH3: Val**, swanmatch:SpacerHole, F.Cu at (140.5, 63.8)
- added RefH4: Val**, swanmatch:SpacerHole, F.Cu at (64.3, 83.8)
- added RefH5: Val**, swanmatch:SpacerHole, F.Cu at (216.7, 83.8)
- C1, C2, C3, C4, C5, C6, C7, J1, J2, J3, J4, J5, J6, R1, R2, R3, R4, U1, Y1: moved to F.Cu
- USB1: footprint Connector_JST:JST_EH_S4B-EH_1x04_P2.50mm_Horizontal -> Connector_PinHeader_2.54mm:PinHeader_1x04_P2.54mm_Horizontal
- moved J4 95.2 mm to (95.3, 21.1)
- moved J1 93.5 mm to (90.3, 21.1)
- moved J2 93.3 mm to (87.8, 21.1)
- moved J3 93.0 mm to (85.3, 21.1)
- moved D41 92.9 mm to (209.6, 95.2), turned to 90 degrees
- moved J5 92.7 mm to (92.8, 21.1)
- moved J6 92.7 mm to (82.8, 21.1)
- moved R2 75.5 mm to (68.1, 24.6)
- moved R3 75.0 mm to (69.9, 21.6)
- moved USB1 73.1 mm to (63.1, 16.6), turned to 180 degrees
- moved SW_R4C1_1 71.4 mm to (104.8, 92.9)
- moved SW_R4C4_1 71.4 mm to (176.2, 92.9)
- moved D38 48.2 mm to (116.7, 95.2), turned to 90 degrees
- moved C7 30.6 mm to (26.8, 94.9)
- moved C6 25.7 mm to (29.3, 94.9)
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- renumbered J4 to JH1
Connections:
- U1 pad 10: col2 -> col11
- U1 pad 11: col3 -> col12
- U1 pad 12: col7 -> col9
- U1 pad 20: col10 -> Net-(U1-Pad20)
- U1 pad 21: col11 -> Net-(U1-Pad21)
- U1 pad 25: col12 -> col1
- U1 pad 26: Net-(U1-Pad26) -> col2
- U1 pad 27: Net-(U1-Pad27) -> col3
- U1 pad 28: col4 -> col7
- U1 pad 29: col5 -> col8
- U1 pad 30: col6 -> row2
- U1 pad 31: col8 -> row1
- U1 pad 32: col9 -> row0
- U1 pad 36: row3 -> col0
- U1 pad 37: row2 -> col4
- U1 pad 38: row1 -> col5
- U1 pad 39: row0 -> col6
- U1 pad 8: col0 -> row3
- U1 pad 9: col1 -> col10
- USB1 pad 1: +5V -> Net-(F1-Pad1)
Routing:
- net row0: track 0.00 -> 356.8 mm, vias 0 -> 3
- net row1: track 0.00 -> 334.5 mm, vias 0 -> 3
- net col11: track 0.00 -> 316.3 mm, vias 0 -> 7
- net col10: track 0.00 -> 296.5 mm, vias 0 -> 7
- net col12: track 0.00 -> 281.0 mm, vias 0 -> 3
- net row2: track 0.00 -> 264.9 mm, vias 0 -> 1
- net col9: track 0.00 -> 233.6 mm, vias 0 -> 7
- net row3: track 0.00 -> 177.2 mm, vias 0 -> 1
- net Net-(J2-Pad1): track 0.00 -> 163.9 mm, vias 0 -> 2
- net col1: track 0.00 -> 131.9 mm, vias 0 -> 7
- net GND: track 139.6 -> 265.6 mm, vias 0 -> 3
- net col2: track 0.00 -> 93.5 mm, vias 0 -> 5
- net col0: track 0.00 -> 92.4 mm, vias 0 -> 4
- net +5V: track 139.5 -> 224.5 mm
- net col3: track 0.00 -> 80.6 mm, vias 0 -> 4
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Other:
- board size 267.7 x 100.7 mm -> 267.7 x 107.7 mm
- net class Default: via_dia 0.8 -> 0.6
- net class GND: trace_width 0.3 -> 0.5
- net class VCC: trace_width 0.3 -> 0.5

Commit message: create pcb done
Parts:
- C1, C2, C3, C4, C5, C6, C7, D42, D43, F1, R1, R2, R3, R4, U1: moved to B.Cu
- D1, D10, D11, D12, D13, D14, D15, D16, D17, D18, D19, D2, D20, D21, D22, D23, D24, D25, D26, D27, D28, D29, D3, D30, D31, D32, D33, D34, D35, D36, D37, D38, D39, D4, D40, D41, D5, D6, D7, D8, D9: footprint swanmatch:D3_SMD_v2 -> mikamo3:D3_SMD_1side
- Y1: value Crystal -> Crystal_GND24_Small; moved to B.Cu
- moved R4 120.1 mm to (146.3, 22.1), turned to 90 degrees
- moved C7 110.5 mm to (109.2, 21.2), turned to 90 degrees
- moved U1 110.0 mm to (135.5, 20.1)
- moved C3 109.6 mm to (120.0, 21.3)
- moved C4 103.3 mm to (106.6, 21.2), turned to 90 degrees
- moved C5 103.3 mm to (104.1, 21.2), turned to 90 degrees
- moved C6 103.3 mm to (101.6, 21.2), turned to 90 degrees
- moved C1 100.6 mm to (127.7, 12.3), turned to 315 degrees
- moved Y1 97.6 mm to (125.2, 15.0), turned to 225 degrees
- moved C2 94.5 mm to (122.5, 17.5), turned to 135 degrees
- moved R1 92.9 mm to (114.1, 20.1)
- moved D43 20.9 mm to (58.3, 16.1)
- moved D42 19.2 mm to (58.3, 24.9)
- moved F1 18.2 mm to (53.6, 13.6)
- moved R3 11.9 mm to (58.3, 19.1)
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Connections:
- U1 pad 1: Net-(U1-Pad1) -> col0
- U1 pad 10: col11 -> row1
- U1 pad 11: col12 -> row0
- U1 pad 12: col9 -> Net-(U1-Pad12)
- U1 pad 25: col1 -> col12
- U1 pad 26: col2 -> Net-(U1-Pad26)
- U1 pad 27: col3 -> Net-(U1-Pad27)
- U1 pad 28: col7 -> col11
- U1 pad 29: col8 -> col10
- U1 pad 30: row2 -> col9
- U1 pad 31: row1 -> col8
- U1 pad 32: row0 -> col7
- U1 pad 36: col0 -> col6
- U1 pad 37: col4 -> col5
- U1 pad 38: col5 -> col4
- U1 pad 39: col6 -> col3
- U1 pad 40: Net-(U1-Pad40) -> col2
- U1 pad 41: Net-(U1-Pad41) -> col1
- U1 pad 9: col10 -> row2
Routing:
- net col2: track 93.5 -> 328.3 mm, vias 5 -> 4
- net row2: track 264.9 -> 496.2 mm, vias 1 -> 14
- net col3: track 80.6 -> 308.2 mm, vias 4 -> 3
- net row3: track 177.2 -> 392.8 mm, vias 1 -> 9
- net col1: track 131.9 -> 337.5 mm, vias 7 -> 4
- net col0: track 92.4 -> 278.4 mm, vias 4 -> 3
- net col12: track 281.0 -> 123.8 mm, vias 3 -> 0
- net col8: track 47.6 -> 143.9 mm, vias 4 -> 2
- net col4: track 47.6 -> 141.3 mm, vias 4 -> 2
- net col5: track 47.4 -> 123.9 mm, vias 4 -> 2
- net row0: track 356.8 -> 426.1 mm, vias 3 -> 24
- net row1: track 334.5 -> 397.3 mm, vias 3 -> 18
- net col9: track 233.6 -> 175.1 mm, vias 7 -> 2
- net col7: track 47.7 -> 102.2 mm, vias 4 -> 2
- net col10: track 296.5 -> 245.8 mm, vias 7 -> 3
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- added copper zone on B.Cu, net GND
- added copper zone on F.Cu, net GND
Other:
- board size 267.7 x 107.7 mm -> 267.7 x 112.7 mm

Commit message: :sparkles: (pcb) fix chore
Parts:
- D42, D43: footprint Diode_SMD:D_SOD-123 -> mikamo3:D_SOD-123-Zener
- Y1: value Crystal_GND24_Small -> Crystal
- moved C4 8.30 mm to (114.9, 21.0)
- moved C5 8.30 mm to (112.4, 21.0)
- moved C6 8.30 mm to (109.9, 21.0)
- moved C7 8.30 mm to (117.5, 21.0)
- moved C3 7.71 mm to (118.7, 13.7), turned to 0 degrees
- moved R1 4.38 mm to (113.5, 15.8)
- moved R4 2.76 mm to (148.6, 20.5)
- moved C1 0.81 mm to (127.6, 13.1)
- moved C2 0.81 mm to (122.4, 18.3)
- moved Y1 0.81 mm to (125.1, 15.8)
- turned SW_RESET1 to 0 degrees
Connections:
- J1 pad 1: col1 -> col2
- J3 pad 1: col2 -> col1
- J4 pad 1: col3 -> col0
- U1 pad 1: col0 -> row0
- U1 pad 10: row1 -> col1
- U1 pad 11: row0 -> col0
- U1 pad 39: col3 -> row3
- U1 pad 40: col2 -> row2
- U1 pad 41: col1 -> row1
- U1 pad 8: row3 -> col3
- U1 pad 9: row2 -> col2
Routing:
- net row3: track 392.8 -> 221.4 mm, vias 9 -> 5
- net row2: track 496.2 -> 357.4 mm
- net row0: track 426.1 -> 321.7 mm, vias 24 -> 14
- net col3: track 308.2 -> 224.9 mm, vias 3 -> 6
- net col11: track 292.5 -> 209.8 mm, vias 5 -> 4
- net col2: track 328.3 -> 248.6 mm, vias 4 -> 6
- net col1: track 337.5 -> 261.1 mm, vias 4 -> 5
- net col10: track 245.8 -> 172.5 mm, vias 3 -> 0
- net row1: track 397.3 -> 335.5 mm, vias 18 -> 14
- net col9: track 175.1 -> 121.4 mm, vias 2 -> 0
- net col8: track 143.9 -> 102.7 mm, vias 2 -> 0
- net Net-(D12-Pad2): track 36.7 -> 65.4 mm
- net col0: track 278.4 -> 300.1 mm, vias 3 -> 2
- net col7: track 102.2 -> 88.1 mm
- net GND: track 311.7 -> 298.0 mm
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Other:
- outline, holes or cut-outs redrawn
- board text added: "D+"
- board text added: "D-"
- board text added: "GND"
- board text added: "VCC"
- board text added: "manaita v1.0 PCB designed by kamo"

Commit message: :sparkles: (all) add plate and fix pcb
Parts:
- removed the RefH1 at (59.5, 44.7)
- removed RefH2, RefH4, RefH5: Val**, swanmatch:SpacerHole
- added RefH1: Val**, swanmatch:SpacerHole, F.Cu at (155.1, 23.2)
- added RefH1: Val**, swanmatch:SpacerHole, F.Cu at (140.9, 101.4)
- added RefH1: Val**, swanmatch:SpacerHole, F.Cu at (26.4, 93.9)
- added RefH1: Val**, swanmatch:SpacerHole, F.Cu at (264.1, 93.9)
- added RefH1: Val**, swanmatch:SpacerHole, F.Cu at (264.1, 23.2)
- added RefH1: Val**, swanmatch:SpacerHole, F.Cu at (26.4, 23.2)
- added USB2: molex_47642-0001, kagizaraya:47642-0001_HandSoldering, F.Cu at (45.3, 15.8)
- D42, D43: footprint mikamo3:D_SOD-123-Zener -> Diode_SMD:D_SOD-123; moved to F.Cu
- F1, R2, R3: moved to F.Cu
- U1: value ATmega32U4-AU -> ATmega32U4
- moved SW_RESET1 102.4 mm to (85.6, 16.1), turned to 180 degrees
- moved D43 12.1 mm to (48.5, 23.2), turned to 180 degrees
- moved D42 10.0 mm to (48.4, 26.3), turned to 180 degrees
- moved USB1 8.97 mm to (61.3, 19.1)
- moved R2 4.61 mm to (54.6, 24.9)
- moved R3 4.51 mm to (54.6, 21.8)
- moved D37 3.48 mm to (266.1, 81.2)
- moved C2 3.21 mm to (123.4, 15.3), turned to 90 degrees
- moved F1 3.03 mm to (56.5, 14.6)
- moved C1 3.01 mm to (129.7, 15.3), turned to 90 degrees
- moved U1 2.42 mm to (136.5, 22.3)
- moved C3 2.33 mm to (120.4, 15.3), turned to 90 degrees
- moved D36 1.77 mm to (266.1, 69.7)
- moved Y1 1.44 mm to (126.5, 15.7), turned to 270 degrees
- moved R4 1.20 mm to (149.8, 20.5)
Connections:
- net Net-(F1-Pad1) renamed VCC
- U1 pad 12: Net-(U1-Pad12) -> (no net)
- U1 pad 18: Net-(U1-Pad18) -> (no net)
- U1 pad 19: Net-(U1-Pad19) -> (no net)
- U1 pad 20: Net-(U1-Pad20) -> (no net)
- U1 pad 21: Net-(U1-Pad21) -> (no net)
- U1 pad 22: Net-(U1-Pad22) -> (no net)
- U1 pad 26: Net-(U1-Pad26) -> (no net)
- U1 pad 27: Net-(U1-Pad27) -> (no net)
- U1 pad 42: Net-(U1-Pad42) -> (no net)
Routing:
- net Net-(J2-Pad1): track 211.8 -> 47.4 mm
- net GND: track 298.0 -> 191.1 mm, vias 0 -> 10
- net D+: track 7.06 -> 24.7 mm, vias 0 -> 1
- net VCC: track 3.26 -> 20.5 mm
- net col0: track 300.1 -> 284.8 mm
- net D-: track 7.29 -> 21.4 mm
- net Net-(D37-Pad2): track 29.2 -> 18.0 mm
- net Net-(D41-Pad2): track 67.0 -> 59.6 mm
- net row3: track 221.4 -> 227.4 mm, vias 5 -> 3
- net +5V: track 180.6 -> 175.0 mm, vias 6 -> 5
- net col5: track 128.1 -> 122.9 mm
- net Net-(R3-Pad1): track 83.3 -> 88.5 mm, vias 0 -> 1
- net row0: track 321.7 -> 325.9 mm, vias 14 -> 15
- net row2: track 357.4 -> 354.2 mm
- net col4: track 143.1 -> 140.4 mm
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Other:
- outline, holes or cut-outs redrawn

Commit message: :sparkles: (all) last fix before create pcb
Parts:
- added D44: LED, LED_SMD:LED_1206_3216Metric_Pad1.42x1.75mm_HandSolder, B.Cu at (99.2, 22.4)
- added R5: 220, Resistor_SMD:R_1206_3216Metric_Pad1.30x1.75mm_HandSolder, B.Cu at (104.8, 22.4)
- D42, D43: footprint Diode_SMD:D_SOD-123 -> mikamo3:D_SOD-123-Zener
Routing:
- net col5: track 122.9 -> 116.0 mm, vias 5 -> 2
- net row0: track 325.9 -> 332.8 mm
- net GND: track 191.1 -> 197.7 mm, vias 10 -> 13
- net row2: track 354.2 -> 358.4 mm, vias 14 -> 13
- net col7: track 85.6 -> 81.5 mm, vias 2 -> 0
- net Net-(R3-Pad1): track 88.5 -> 84.5 mm
- net col1: track 262.6 -> 266.0 mm
- net col3: track 222.8 -> 225.9 mm, vias 6 -> 4
- net +5V: track 175.0 -> 177.9 mm, vias 5 -> 6
- net row3: track 227.4 -> 230.0 mm
- net Net-(D44-Pad2): track 0.00 -> 2.55 mm
- net Net-(C3-Pad1): track 20.4 -> 22.2 mm
- net col10: track 171.8 -> 173.3 mm
- net col4: track 140.4 -> 139.0 mm, vias 7 -> 5
- net Net-(D41-Pad2): track 59.6 -> 61.0 mm
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