File: pcb/manaita.sch (KiCad schematic (older format))
At the start: 110 parts, among them J1 SCK, J2 RST, J3 MOSI, J4 MISO, J5 VCC, J6 GND, U1 ATmega32U4-AU, Y1 Crystal_GND24_Small

Commit message: :sparkles: (all) add plate and fix pcb
Parts:
- added USB2: molex_47642-0001, kagizaraya:47642-0001_HandSoldering, symbol mikamo3:molex_47642-0001
Connections:
- net D+: now also USB2.3 (D+)
- net D-: now also USB2.2 (D-)
- net GND: now also USB2.5 (GND), USB2.6 (Sield)
- net VCC: now reaches F1.1, USB1.1 (Pin_1)
- net VCC: now also USB2.1 (VCC)
- no-connect marks 9 -> 10
Other:
- moved on the sheet: F1, USB1
Changed lines of the file:
@@
 NoConn ~ 5650 4000
-$Comp
-L power:PWR_FLAG #FLG01
-U 1 1 5FB94B54
-P 1900 5400
-F 0 "#FLG01" H 1900 5475 50  0001 C CNN
-F 1 "PWR_FLAG" H 1900 5573 50  0000 C CNN
-F 2 "" H 1900 5400 50  0001 C CNN
-F 3 "~" H 1900 5400 50  0001 C CNN
-	1    1900 5400
-	-1   0    0    1
-$EndComp
-$Comp
-L power:+5V #PWR08
-U 1 1 5FB93BB3
-P 1900 5400
-F 0 "#PWR08" H 1900 5250 50  0001 C CNN
-F 1 "+5V" H 1915 5573 50  0000 C CNN
-F 2 "" H 1900 5400 50  0001 C CNN
-F 3 "" H 1900 5400 50  0001 C CNN
-	1    1900 5400
-	1    0    0    -1
-$EndComp
 $Comp
 L Connector_Generic:Conn_01x04 USB1
 U 1 1 5FCC7385
-P 2100 5950
-F 0 "USB1" H 2180 5942 50  0000 L CNN
-F 1 "Conn_01x04" H 2180 5851 50  0000 L CNN
-F 2 "Connector_PinHeader_2.54mm:PinHeader_1x04_P2.54mm_Horizontal" H 2100 5950 50  0001 C CNN
-F 3 "~" H 2100 5950 50  0001 C CNN
-	1    2100 5950
-	1    0    0    -1
-$EndComp
-Text GLabel 1900 6050 0    50   Input ~ 0
-D+
-Text GLabel 1900 5950 0    50   Input ~ 0
-D-
+P 1550 5750
+F 0 "USB1" H 1630 5742 50  0000 L CNN
+F 1 "Conn_01x04" H 1630 5651 50  0000 L CNN
+F 2 "Connector_PinHeader_2.54mm:PinHeader_1x04_P2.54mm_Horizontal" H 1550 5750 50  0001 C CNN
+F 3 "~" H 1550 5750 50  0001 C CNN
+	1    1550 5750
+	-1   0    0    1
+$EndComp
 $Comp
 L power:+5V #PWR011
 U 1 1 5FCD6AFB
-P 1700 5850
-F 0 "#PWR011" H 1700 5700 50  0001 C CNN
-F 1 "+5V" H 1715 6023 50  0000 C CNN
-F 2 "" H 1700 5850 50  0001 C CNN
-F 3 "" H 1700 5850 50  0001 C CNN
-	1    1700 5850
-	0    -1   -1   0
+P 3100 5850
+F 0 "#PWR011" H 3100 5700 50  0001 C CNN
+F 1 "+5V" H 3115 6023 50  0000 C CNN
+F 2 "" H 3100 5850 50  0001 C CNN
+F 3 "" H 3100 5850 50  0001 C CNN
+	1    3100 5850
+	0    1    1    0
 $EndComp
 $Comp
 L power:GND #PWR013
 U 1 1 5FCD798D
-P 1900 6150
-F 0 "#PWR013" H 1900 5900 50  0001 C CNN
-F 1 "GND" H 1905 5977 50  0000 C CNN
-F 2 "" H 1900 6150 50  0001 C CNN
-F 3 "" H 1900 6150 50  0001 C CNN
-	1    1900 6150
-	0    1    1    0
-$EndComp
-$Comp
-L power:PWR_FLAG #FLG02
-U 1 1 5FCF83A3
-P 2250 5400
-F 0 "#FLG02" H 2250 5475 50  0001 C CNN
-F 1 "PWR_FLAG" H 2250 5573 50  0000 C CNN
-F 2 "" H 2250 5400 50  0001 C CNN
-F 3 "~" H 2250 5400 50  0001 C CNN
-	1    2250 5400
-	-1   0    0    1
-$EndComp
-$Comp
-L power:GND #PWR09
-U 1 1 5FCF8CE0
-P 2250 5400
-F 0 "#PWR09" H 2250 5150 50  0001 C CNN
-F 1 "GND" H 2255 5227 50  0000 C CNN
-F 2 "" H 2250 5400 50  0001 C CNN
-F 3 "" H 2250 5400 50  0001 C CNN
-	1    2250 5400
-	-1   0    0    1
+P 3150 5550
+F 0 "#PWR013" H 3150 5300 50  0001 C CNN
+F 1 "GND" H 3155 5377 50  0000 C CNN
+F 2 "" H 3150 5550 50  0001 C CNN
+F 3 "" H 3150 5550 50  0001 C CNN
+	1    3150 5550
+	0    -1   -1   0
 $EndComp
 $Comp
@@
 	3200 4100 2400 4100
 Connection ~ 3200 4100
-Wire Wire Line
-	2400 4100 1600 4100
 Connection ~ 2400 4100
 Wire Wire Line
@@
 L Device:Polyfuse_Small F1
 U 1 1 5FC7B42C
-P 1800 5850
-F 0 "F1" V 1595 5850 50  0000 C CNN
-F 1 "500mA" V 1686 5850 50  0000 C CNN
-F 2 "Fuse:Fuse_0805_2012Metric_Pad1.15x1.40mm_HandSolder" H 1850 5650 50  0001 L CNN
-F 3 "~" H 1800 5850 50  0001 C CNN
-	1    1800 5850
-	0    1    1    0
+P 2550 5850
+F 0 "F1" V 2345 5850 50  0000 C CNN
+F 1 "500mA" V 2436 5850 50  0000 C CNN
+F 2 "Fuse:Fuse_0805_2012Metric_Pad1.15x1.40mm_HandSolder" H 2600 5650 50  0001 L CNN
+F 3 "~" H 2550 5850 50  0001 C CNN
+	1    2550 5850
+	0    -1   -1   0
 $EndComp
 $Comp
@@
 Wire Wire Line
 	7700 3700 7950 3700
+$Comp
+L power:PWR_FLAG #FLG0102
+U 1 1 5FE7E5EF
+P 4900 6700
+F 0 "#FLG0102" H 4900 6775 50  0001 C CNN
+F 1 "PWR_FLAG" H 4900 6873 50  0000 C CNN
+F 2 "" H 4900 6700 50  0001 C CNN
+F 3 "~" H 4900 6700 50  0001 C CNN
+	1    4900 6700
+	1    0    0    -1
+$EndComp
+Wire Wire Line
+	2650 5850 3100 5850
+$Comp
+L power:GND #PWR0104
+U 1 1 5FECCFAF
+P 4900 6700
+F 0 "#PWR0104" H 4900 6450 50  0001 C CNN
+F 1 "GND" H 4905 6527 50  0000 C CNN
+F 2 "" H 4900 6700 50  0001 C CNN
+F 3 "" H 4900 6700 50  0001 C CNN
+	1    4900 6700
+	1    0    0    -1
+$EndComp
+Wire Wire Line
+	1750 5550 2550 5550
+Wire Wire Line
+	1750 5850 1850 5850
+Wire Wire Line
+	2400 4100 1600 4100
+$Comp
+L mikamo3:molex_47642-0001 USB2
+U 1 1 60090139
+P 1700 5350
+F 0 "USB2" H 1472 4959 50  0000 R CNN
+F 1 "molex_47642-0001" H 1472 5050 50  0000 R CNN
+F 2 "kagizaraya:47642-0001_HandSoldering" H 1700 5350 50  0001 C CNN
+F 3 "" H 1700 5350 50  0001 C CNN
+	1    1700 5350
+	1    0    0    1
+$EndComp
+Wire Wire Line
+	2050 4750 2050 4850
+NoConn ~ 2050 4950
+Text GLabel 2600 5650 2    50   Input ~ 0
+D+
+Text GLabel 2600 5750 2    50   Input ~ 0
+D-
+Wire Wire Line
+	1750 5750 2250 5750
+Wire Wire Line
+	1750 5650 2400 5650
+Wire Wire Line
+	2050 5250 2050 5850
+Connection ~ 2050 5850
+Wire Wire Line
+	2050 5850 2450 5850
+Wire Wire Line
+	2050 5150 2250 5150
+Wire Wire Line
+	2250 5150 2250 5750
+Connection ~ 2250 5750
+Wire Wire Line
+	2250 5750 2600 5750
+Wire Wire Line
+	2050 5050 2400 5050
+Wire Wire Line
+	2400 5050 2400 5650
+Connection ~ 2400 5650
+Wire Wire Line
+	2400 5650 2600 5650
+Wire Wire Line
+	2050 4850 2550 4850
+Wire Wire Line
+	2550 4850 2550 5550
+Connection ~ 2050 4850
+Connection ~ 2550 5550
+Wire Wire Line
+	2550 5550 3150 5550
+$Comp
+L power:VCC #PWR0105
+U 1 1 6019E274
+P 1850 5850
+F 0 "#PWR0105" H 1850 5700 50  0001 C CNN
+F 1 "VCC" H 1865 6023 50  0000 C CNN
+F 2 "" H 1850 5850 50  0001 C CNN
+F 3 "" H 1850 5850 50  0001 C CNN
+	1    1850 5850
+	-1   0    0    1
+$EndComp
+Connection ~ 1850 5850
+Wire Wire Line
+	1850 5850 2050 5850
+$Comp
+L power:PWR_FLAG #FLG0103
+U 1 1 6019EB2C
+P 4000 6700
+F 0 "#FLG0103" H 4000 6775 50  0001 C CNN
+F 1 "PWR_FLAG" H 4000 6873 50  0000 C CNN
+F 2 "" H 4000 6700 50  0001 C CNN
+F 3 "~" H 4000 6700 50  0001 C CNN
+	1    4000 6700
+	1    0    0    -1
+$EndComp
+$Comp
+L power:VCC #PWR0106
+U 1 1 6019F1C4
+P 4000 6700
+F 0 "#PWR0106" H 4000 6550 50  0001 C CNN
+F 1 "VCC" H 4015 6873 50  0000 C CNN
+F 2 "" H 4000 6700 50  0001 C CNN
+F 3 "" H 4000 6700 50  0001 C CNN
+	1    4000 6700
+	-1   0    0    1
+$EndComp
+$Comp
+L power:+5V #PWR0103
+U 1 1 5FFE47A9
+P 4500 6700
+F 0 "#PWR0103" H 4500 6550 50  0001 C CNN
+F 1 "+5V" H 4515 6873 50  0000 C CNN
+F 2 "" H 4500 6700 50  0001 C CNN
+F 3 "" H 4500 6700 50  0001 C CNN
+	1    4500 6700
+	-1   0    0    1
+$EndComp
+$Comp
+L power:PWR_FLAG #FLG0101
+U 1 1 5FE38672
+P 4500 6700
+F 0 "#FLG0101" H 4500 6775 50  0001 C CNN
+F 1 "PWR_FLAG" H 4500 6873 50  0000 C CNN
+F 2 "" H 4500 6700 50  0001 C CNN
+F 3 "~" H 4500 6700 50  0001 C CNN
+	1    4500 6700
+	1    0    0    -1
+$EndComp
 $EndSCHEMATC

Commit message: :sparkles: (all) last fix before create pcb
Parts:
- added D44: LED, LED_SMD:LED_1206_3216Metric_Pad1.42x1.75mm_HandSolder, symbol Device:LED
- added R5: 220, Resistor_SMD:R_1206_3216Metric_Pad1.30x1.75mm_HandSolder, symbol Device:R_Small
Changed lines of the file:
@@
+	1    0    0    -1
+$EndComp
+$Comp
+L power:+5V #PWR08
+U 1 1 5FD871F9
+P 3100 6650
+F 0 "#PWR08" H 3100 6500 50  0001 C CNN
+F 1 "+5V" H 3115 6823 50  0000 C CNN
+F 2 "" H 3100 6650 50  0001 C CNN
+F 3 "" H 3100 6650 50  0001 C CNN
+	1    3100 6650
+	1    0    0    -1
+$EndComp
+$Comp
+L Device:LED D44
+U 1 1 5FD881AF
+P 3100 7000
+F 0 "D44" V 3139 6882 50  0000 R CNN
+F 1 "LED" V 3048 6882 50  0000 R CNN
+F 2 "LED_SMD:LED_1206_3216Metric_Pad1.42x1.75mm_HandSolder" H 3100 7000 50  0001 C CNN
+F 3 "~" H 3100 7000 50  0001 C CNN
+	1    3100 7000
+	0    -1   -1   0
+$EndComp
+$Comp
+L Device:R_Small R5
+U 1 1 5FD8B726
+P 3100 6750
+F 0 "R5" V 2904 6750 50  0000 C CNN
+F 1 "220" V 2995 6750 50  0000 C CNN
+F 2 "Resistor_SMD:R_1206_3216Metric_Pad1.30x1.75mm_HandSolder" V 3030 6750 50  0001 C CNN
+F 3 "~" H 3100 6750 50  0001 C CNN
+	1    3100 6750
+	-1   0    0    1
+$EndComp
+$Comp
+L power:GND #PWR09
+U 1 1 5FD963AE
+P 3100 7150
+F 0 "#PWR09" H 3100 6900 50  0001 C CNN
+F 1 "GND" H 3105 6977 50  0000 C CNN
+F 2 "" H 3100 7150 50  0001 C CNN
+F 3 "" H 3100 7150 50  0001 C CNN
+	1    3100 7150
 	1    0    0    -1
 $EndComp
