File: pcb/manaita_topplate.kicad_pcb (KiCad board)
At the start: 2 copper layers, 267.6 x 112.7 mm, 7 parts, among them J4 Conn_01x01

Commit message: :sparkles: (all) last fix before create pcb
Other:
- outline, holes or cut-outs redrawn
