File: v2/main/main.kicad_pcb (KiCad board)
At the start: 2 copper layers, 247.6 x 76.2 mm, 90 parts, among them SW1 SW_PUSH, SW10 SW_PUSH, SW11 SW_PUSH, SW12 SW_PUSH, SW13 SW_PUSH, SW14 SW_PUSH, SW15 SW_PUSH, SW16 SW_PUSH, SW17 SW_PUSH, SW18 SW_PUSH, SW19 SW_PUSH, SW2 SW_PUSH, SW20 SW_PUSH, SW21 SW_PUSH, SW22 SW_PUSH, SW23 SW_PUSH, SW24 SW_PUSH, SW25 SW_PUSH, SW26 SW_PUSH, SW27 SW_PUSH, SW28 SW_PUSH, SW29 SW_PUSH, SW3 SW_PUSH, SW30 SW_PUSH, SW31 SW_PUSH, SW32 SW_PUSH, SW33 SW_PUSH, SW34 SW_PUSH, SW35 SW_PUSH, SW36 SW_PUSH, SW37 SW_PUSH, SW38 SW_PUSH, SW39 SW_PUSH, SW4 SW_PUSH, SW40 SW_PUSH, SW41 SW_PUSH, SW42 SW_PUSH, SW43 SW_PUSH, SW44 SW_PUSH, SW45 SW_PUSH, SW5 SW_PUSH, SW6 SW_PUSH, SW7 SW_PUSH, SW8 SW_PUSH, SW9 SW_PUSH

Commit message: Add initial KiCad project files for version 2
- Created top.kicad_pro with board design settings, rules, and dimensions.
- Added top.kicad_sch with basic schematic structure and metadata.
Parts:
- added C1: 100n, Capacitor_SMD:C_0402_1005Metric, B.Cu at (267.1, 56.8)
- added C10: 100n, Capacitor_SMD:C_0402_1005Metric, B.Cu at (274.2, 39.5)
- added C11: 15p, Capacitor_SMD:C_0603_1608Metric, B.Cu at (257.0, 32.8)
- added C12: 1u, Capacitor_SMD:C_0402_1005Metric, B.Cu at (271.2, 32.4)
- added C13: 1u, Capacitor_SMD:C_0402_1005Metric, B.Cu at (272.5, 30.3)
- added C14: 15p, Capacitor_SMD:C_0603_1608Metric, B.Cu at (251.0, 32.8)
- added C15: 10u, Capacitor_SMD:C_0805_2012Metric, B.Cu at (274.6, 48.5)
- added C16: 10u, Capacitor_SMD:C_0805_2012Metric, B.Cu at (274.1, 62.7)
- added C2: 100n, Capacitor_SMD:C_0402_1005Metric, B.Cu at (272.0, 39.5)
- added C3: 100n, Capacitor_SMD:C_0402_1005Metric, B.Cu at (259.5, 32.7)
- added C4: 100n, Capacitor_SMD:C_0402_1005Metric, B.Cu at (269.2, 41.0)
- added C5: 100n, Capacitor_SMD:C_0402_1005Metric, B.Cu at (262.8, 46.9)
- added C6: 100n, Capacitor_SMD:C_0402_1005Metric, B.Cu at (272.5, 31.4)
- added C7: 100n, Capacitor_SMD:C_0402_1005Metric, B.Cu at (256.2, 28.8)
- added C8: 100n, Capacitor_SMD:C_0402_1005Metric, B.Cu at (254.7, 28.8)
- added C9: 100n, Capacitor_SMD:C_0402_1005Metric, B.Cu at (273.1, 39.5)
- added J1: USB_C_Receptacle_USB2.0_14P, Connector_USB:USB_C_Receptacle_Palconn_UTC16-G, B.Cu at (152.6, 15.5)
- added R1: DNF, Resistor_SMD:R_0402_1005Metric, B.Cu at (263.0, 58.6)
- added R2: 1k, Resistor_SMD:R_0402_1005Metric, B.Cu at (257.2, 58.6)
- added R3: 1k, Resistor_SMD:R_0402_1005Metric, B.Cu at (253.5, 30.5)
- added R4: 27, Resistor_SMD:R_0603_1608Metric, B.Cu at (271.7, 35.6)
- added R5: 27, Resistor_SMD:R_0603_1608Metric, B.Cu at (271.7, 33.7)
- added R6: 5.1k, Resistor_SMD:R_0402_1005Metric, B.Cu at (147.8, 20.1)
- added R7: 5.1k, Resistor_SMD:R_0402_1005Metric, B.Cu at (149.1, 20.1)
- added R8: 10k, Resistor_SMD:R_0402_1005Metric, B.Cu at (246.8, 88.3)
- added SW46: BOOT, kamo3_footprint:Tact_Switch_5.1_5.1mm_SMD, B.Cu at (252.2, 91.7)
- added SW47: RUN, kamo3_footprint:Tact_Switch_5.1_5.1mm_SMD, B.Cu at (243.0, 91.7)
- added U1: W25Q128JVS, Package_SO:SOIC-8_5.23x5.23mm_P1.27mm, B.Cu at (261.3, 55.0)
- added U2: NCP1117-3.3_SOT223, Package_TO_SOT_SMD:SOT-223-3_TabPin2, B.Cu at (272.6, 55.1)
- added U3: RP2040, rp2040:RP2040-QFN-56, B.Cu at (265.1, 35.8)
- added Y1: ABM8-272-T3, Crystal:Crystal_SMD_3225-4Pin_3.2x2.5mm, B.Cu at (254.1, 32.9)
- D1, D10, D11, D12, D13, D14, D15, D16, D17, D18, D19, D2, D20, D21, D22, D23, D24, D25, D26, D27, D28, D29, D3, D30, D31, D32, D33, D34, D35, D36, D37, D38, D39, D4, D40, D41, D42, D43, D44, D45, D5, D6, D7, D8, D9: moved to B.Cu
- SW41: footprint kamo3_footprint:SW_CherryMX_Hotswap_2.25u -> kamo3_footprint:SW_CherryMX_Hotswap_1.00u
- SW42: footprint kamo3_footprint:SW_CherryMX_Hotswap_2.75u -> kamo3_footprint:SW_CherryMX_Hotswap_1.00u
- moved D26 352.1 mm to (52.4, 67.0), turned to 90 degrees
- moved D14 350.8 mm to (47.6, 47.9), turned to 90 degrees
- moved D1 347.9 mm to (45.3, 28.9), turned to 90 degrees
- moved D38 330.7 mm to (81.0, 86.0), turned to 90 degrees
- moved D15 329.5 mm to (69.1, 47.9), turned to 90 degrees
- moved D2 329.2 mm to (64.3, 28.9), turned to 90 degrees
- moved D27 325.9 mm to (78.6, 67.0), turned to 90 degrees
- moved D16 310.6 mm to (88.1, 47.9), turned to 90 degrees
- moved D3 310.5 mm to (83.3, 28.9), turned to 90 degrees
- moved D28 306.8 mm to (97.6, 67.0), turned to 90 degrees
- moved D39 306.7 mm to (104.8, 86.0), turned to 90 degrees
- moved D4 291.9 mm to (102.4, 28.9), turned to 90 degrees
- moved D17 291.8 mm to (107.2, 47.9), turned to 90 degrees
- moved D29 287.7 mm to (116.7, 67.0), turned to 90 degrees
- moved D40 282.7 mm to (128.6, 86.0), turned to 90 degrees
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Connections:
- net Net-(D1-K) renamed /row0
- net Net-(D14-K) renamed /row1
- net Net-(D26-K) renamed /row2
- net Net-(D38-K) renamed /row3
- net Net-(SW11-Pad1) renamed /col10
- net Net-(SW12-Pad1) renamed /col11
- SW1 pad 1: Net-(SW1-Pad1) -> /col0
- SW10 pad 1: Net-(SW10-Pad1) -> /col9
- SW13 pad 1: unconnected-(SW13-Pad1) -> /col12
- SW14 pad 1: Net-(SW1-Pad1) -> /col0
- SW15 pad 1: Net-(SW15-Pad1) -> /col1
- SW16 pad 1: Net-(SW16-Pad1) -> /col2
- SW17 pad 1: Net-(SW17-Pad1) -> /col3
- SW18 pad 1: Net-(SW18-Pad1) -> /col4
- SW19 pad 1: Net-(SW19-Pad1) -> /col5
- SW2 pad 1: Net-(SW15-Pad1) -> /col1
- SW20 pad 1: Net-(SW20-Pad1) -> /col6
- SW21 pad 1: Net-(SW21-Pad1) -> /col7
- SW22 pad 1: Net-(SW22-Pad1) -> /col8
- SW23 pad 1: Net-(SW10-Pad1) -> /col9
- SW26 pad 1: Net-(SW1-Pad1) -> /col0
- SW27 pad 1: Net-(SW15-Pad1) -> /col1
- SW28 pad 1: Net-(SW16-Pad1) -> /col2
- SW29 pad 1: Net-(SW17-Pad1) -> /col3
- SW3 pad 1: Net-(SW16-Pad1) -> /col2
- SW30 pad 1: Net-(SW18-Pad1) -> /col4
- SW31 pad 1: Net-(SW19-Pad1) -> /col5
- SW32 pad 1: Net-(SW20-Pad1) -> /col6
- SW33 pad 1: Net-(SW21-Pad1) -> /col7
- SW34 pad 1: Net-(SW22-Pad1) -> /col8
- SW35 pad 1: Net-(SW10-Pad1) -> /col9
- SW38 pad 1: Net-(SW1-Pad1) -> /col1
- SW39 pad 1: Net-(SW15-Pad1) -> /col2
- SW4 pad 1: Net-(SW17-Pad1) -> /col3
- SW40 pad 1: Net-(SW16-Pad1) -> /col3
- SW41 pad 1: Net-(SW17-Pad1) -> /col4
- SW42 pad 1: Net-(SW18-Pad1) -> /col5
- SW43 pad 1: Net-(SW19-Pad1) -> /col6
- SW44 pad 1: Net-(SW20-Pad1) -> /col8
- SW45 pad 1: Net-(SW21-Pad1) -> /col9
- SW5 pad 1: Net-(SW18-Pad1) -> /col4
- SW6 pad 1: Net-(SW19-Pad1) -> /col5
- SW7 pad 1: Net-(SW20-Pad1) -> /col6
- SW8 pad 1: Net-(SW21-Pad1) -> /col7
- SW9 pad 1: Net-(SW22-Pad1) -> /col8
Routing:
- net /row2: track 0.00 -> 555.1 mm, vias 0 -> 13
- net /row1: track 0.00 -> 542.4 mm, vias 0 -> 13
- net /row3: track 0.00 -> 527.7 mm, vias 0 -> 2
- net /row0: track 0.00 -> 333.5 mm, vias 0 -> 12
- net /col1: track 0.00 -> 279.2 mm, vias 0 -> 2
- net /col0: track 0.00 -> 278.0 mm, vias 0 -> 2
- net /col2: track 0.00 -> 263.7 mm, vias 0 -> 2
- net /col3: track 0.00 -> 249.2 mm, vias 0 -> 2
- net /col4: track 0.00 -> 232.8 mm, vias 0 -> 2
- net /col5: track 0.00 -> 214.6 mm, vias 0 -> 2
- net /col6: track 0.00 -> 198.6 mm, vias 0 -> 2
- net +3V3: track 0.00 -> 167.6 mm
- net /col8: track 0.00 -> 165.3 mm, vias 0 -> 2
- net VBUS: track 0.00 -> 165.1 mm
- net /col9: track 0.00 -> 150.9 mm, vias 0 -> 2
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- added copper zone on B.Cu, net GND
- added copper zone on F.Cu, net GND
Other:
- board size 247.6 x 76.2 mm -> 249.6 x 91.7 mm
